Commit message: Replace with correct stl
Signed-off-by: Yadunund <yadunund@openrobotics.org>

File: robot_specific_config/abb_crb1100_support/urdf/crb1100_4_58_macro.xacro (robot description, xacro)
@@ -7,53 +7,13 @@
       <visual name="visual">
         <geometry>
-          <mesh filename="package://abb_crb1100_support/meshes/crb1100_4_58/base_link.dae"/>
+          <mesh filename="package://abb_crb1100_support/meshes/crb1100_4_58/base_link.stl"/>
         </geometry>
         <xacro:material_abb_white />
       </visual>
-      <collision name="Base_Box001">
-        <pose>-0.00780786 0.000316538 0.006 0.0 0.0 0.0</pose>
+      <collision name"collision">
         <geometry>
-          <box>
-            <size>0.174 0.158 0.012</size>
-          </box>
-          <xacro:material_abb_yellow />
+          <mesh filename="package://abb_crb1100_support/meshes/crb1100_4_58/base_link.stl"/>
         </geometry>
-      </collision>
-      <collision name="Base_Cylinder001">
-        <pose>0.0 0.0 0.0728 0.0 0.0 0.0</pose>
-        <geometry>
-          <cylinder>
-            <length>0.1456</length>
-            <radius>0.0719661</radius>
-          </cylinder>
-          <xacro:material_abb_yellow />
-        </geometry>
-      </collision>
-      <collision name="Base_Box002">
-        <pose>-0.079843 0.0 0.0749219 1.5708 0.0 -1.5708</pose>
-        <geometry>
-          <box>
-            <size>0.110911 0.139336 0.0984126</size>
-          </box>
-          <xacro:material_abb_yellow />
-        </geometry>
-      </collision>
-      <collision name="Base_Box003">
-        <pose>-0.13596 0.0 0.103253 1.5708 0.0 -1.5708</pose>
-        <geometry>
-          <box>
-            <size>0.0964925 0.0459809 0.0285397</size>
-          </box>
-          <xacro:material_abb_yellow />
-        </geometry>
-      </collision>
-      <collision name="Base_Box004">
-        <pose>-0.131965 0.0 0.045724 1.5708 0.0 -1.5708</pose>
-        <geometry>
-          <box>
-            <size>0.0635693 0.0710773 0.0205486</size>
-          </box>
-          <xacro:material_abb_yellow />
-        </geometry>
+        <xacro:material_abb_yellow />
       </collision>
     </link>
@@ -61,54 +21,13 @@
       <visual>
         <geometry>
-          <mesh filename="package://abb_crb1100_support/meshes/crb1100_4_58/link_1.dae"/>
+          <mesh filename="package://abb_crb1100_support/meshes/crb1100_4_58/link_1.stl"/>
         </geometry>
         <xacro:material_abb_white />
       </visual>
-      <collision name="Link1_Cylinder002">
-        <pose>0.0 0.0 0.180716 0.0 0.0 0.0</pose>
+      <collision name="collision">
         <geometry>
-          <cylinder>
-            <length>0.0695336</length>
-            <radius>0.0880028</radius>
-          </cylinder>
-          <xacro:material_abb_yellow />
+          <mesh filename="package://abb_crb1100_support/meshes/crb1100_4_58/link_1.stl"/>
         </geometry>
-      </collision>
-      <collision name="Link1_Cylinder003">
-        <pose>-2.53022e-05 -0.000703648 0.327248 1.5708 0.0 0.0</pose>
-        <geometry>
-          <cylinder>
-            <length>0.184809</length>
-            <radius>0.0517311</radius>
-          </cylinder>
-          <xacro:material_abb_yellow />
-        </geometry>
-      </collision>
-      <collision name="Link1_Box005">
-        <pose>0.00740042 -0.0015163 0.268765 0.0 -0.131547 0.0</pose>
-        <geometry>
-          <box>
-            <size>0.0988751 0.182474 0.12116</size>
-          </box>
-          <xacro:material_abb_yellow />
-        </geometry>
-      </collision>
-      <collision name="Link1_Box006">
-        <pose>-0.0321942 -0.0015163 0.218345 0.0 -0.213012 0.0</pose>
-        <geometry>
-          <box>
-            <size>0.0988751 0.178825 0.0508871</size>
-          </box>
-          <xacro:material_abb_yellow />
-        </geometry>
-      </collision>
-      <collision name="Link1_Box007">
-        <pose>0.0360969 -0.00151631 0.209101 0.0 0.317913 0.0</pose>
-        <geometry>
-          <box>
-            <size>0.0988751 0.164519 0.0783661</size>
-          </box>
-          <xacro:material_abb_yellow />
-        </geometry>
+        <xacro:material_abb_yellow />
       </collision>
     </link>
@@ -116,35 +35,13 @@
       <visual>
         <geometry>
-          <mesh filename="package://abb_crb1100_support/meshes/crb1100_4_58/link_2.dae"/>
+          <mesh filename="package://abb_crb1100_support/meshes/crb1100_4_58/link_2.stl"/>
         </geometry>
         <xacro:material_abb_white />
       </visual>
       <collision name="Link2_Box008">
-        <pose>-0.0174075 0.0 0.423644 0.0 0.0 0.0</pose>
         <geometry>
-          <box>
-            <size>0.0667305 0.0928778 0.198962</size>
-          </box>
-          <xacro:material_abb_yellow />
+          <mesh filename="package://abb_crb1100_support/meshes/crb1100_4_58/link_2.stl"/>
         </geometry>
-      </collision>
-      <collision name="Link2_Cylinder004">
-        <pose>-0.000196304 -0.000291631 0.606764 1.5708 0.0 0.0</pose>
-        <geometry>
-          <cylinder>
-            <length>0.178434</length>
-            <radius>0.0465957</radius>
-          </cylinder>
-          <xacro:material_abb_yellow />
-        </geometry>
-      </collision>
-      <collision name="Link2_Box009">
-        <pose>-0.0103307 0.0 0.531581 0.0 0.01412 0.0</pose>
-        <geometry>
-          <box>
-            <size>0.0734036 0.176468 0.163149</size>
-          </box>
-          <xacro:material_abb_yellow />
-        </geometry>
+        <xacro:material_abb_yellow />
       </collision>
     </link>
@@ -152,55 +49,13 @@
       <visual>
         <geometry>
-          <mesh filename="package://abb_crb1100_support/meshes/crb1100_4_58/link_3.dae"/>
+          <mesh filename="package://abb_crb1100_support/meshes/crb1100_4_58/link_3.stl"/>
         </geometry>
         <xacro:material_abb_white />
       </visual>
-      <collision name="Link3_Cylinder005">
-        <pose>-1.58772e-05 0.0 0.617021 1.5708 0.0 -1.5708</pose>
+      <collision name="collision">
         <geometry>
-          <cylinder>
-            <length>0.146229</length>
-            <radius>0.0454588</radius>
-          </cylinder>
-          <xacro:material_abb_yellow />
+          <mesh filename="package://abb_crb1100_support/meshes/crb1100_4_58/link_3.stl"/>
         </geometry>
-      </collision>
-      <collision name="Link3_Cylinder006">
-        <pose>0.000346811 -6.09569e-05 0.607321 1.5708 0.0 -1.19209e-07</pose>
-        <geometry>
-          <cylinder>
-            <length>0.0954674</length>
-            <radius>0.0454588</radius>
-          </cylinder>
-          <xacro:material_abb_yellow />
-        </geometry>
-      </collision>
-      <collision name="Link3_Cylinder007">
-        <pose>-1.58772e-05 0.0 0.589443 1.5708 0.0 -1.5708</pose>
-        <geometry>
-          <cylinder>
-            <length>0.146229</length>
-            <radius>0.0454588</radius>
-          </cylinder>
-          <xacro:material_abb_yellow />
-        </geometry>
-      </collision>
-      <collision name="Link3_Box010">
-        <pose>-0.0169157 0.0 0.653855 0.0 0.0 0.0</pose>
-        <geometry>
-          <box>
-            <size>0.018736 0.0498875 0.0203162</size>
-          </box>
-          <xacro:material_abb_yellow />
-        </geometry>
-      </collision>
-      <collision name="Link3_Box011">
-        <pose>-0.0289604 -0.0174093 0.565988 0.0 0.0 0.0</pose>
-        <geometry>
-          <box>
-            <size>0.018736 0.0498875 0.0262079</size>
-          </box>
-          <xacro:material_abb_yellow />
-        </geometry>
+        <xacro:material_abb_yellow />
       </collision>
     </link>
@@ -208,63 +63,13 @@
       <visual>
         <geometry>
-          <mesh filename="package://abb_crb1100_support/meshes/crb1100_4_58/link_4.dae"/>
+          <mesh filename="package://abb_crb1100_support/meshes/crb1100_4_58/link_4.stl"/>
         </geometry>
         <xacro:material_abb_white />
       </visual>
-      <collision name="Link4_Cylinder008">
-        <pose>0.15523 0.0 0.617 1.5708 0.0 1.5708</pose>
+      <collision name="collision">
         <geometry>
-          <cylinder>
-            <length>0.163185</length>
-            <radius>0.0452081</radius>
-          </cylinder>
+          <mesh filename="package://abb_crb1100_support/meshes/crb1100_4_58/link_4.stl"/>
         </geometry>
-      </collision>
-      <collision name="Link4_Cylinder009">
-        <pose>0.3 0.0 0.617 1.5708 0.0 -1.74846e-07</pose>
-        <geometry>
-          <cylinder>
-            <length>0.102</length>
-            <radius>0.038</radius>
-          </cylinder>
-          <xacro:material_abb_yellow />
-        </geometry>
-      </collision>
-      <collision name="Link4_Cylinder010">
-        <pose>0.179 0.0 0.617 1.5708 0.0 -1.74846e-07</pose>
-        <geometry>
-          <cylinder>
-            <length>0.102</length>
-            <radius>0.038</radius>
-          </cylinder>
-          <xacro:material_abb_yellow />
-        </geometry>
-      </collision>
-      <collision name="Link4_Box012">
-        <pose>0.239561 0.0 0.617 0.0 0.0 0.0</pose>
-        <geometry>
-          <box>
-            <size>0.12 0.102032 0.076</size>
-          </box>
-          <xacro:material_abb_yellow />
-        </geometry>
-      </collision>
-      <collision name="Link4_Box013">
-        <pose>0.154738 0.0 0.649546 0.0 -0.436332 0.0</pose>
-        <geometry>
-          <box>
-            <size>0.0893911 0.0609485 0.0468981</size>
-          </box>
-          <xacro:material_abb_yellow />
-        </geometry>
-      </collision>
-      <collision name="Link4_Box014">
-        <pose>0.203204 0.0 0.647963 0.0 0.0 0.0</pose>
-        <geometry>
-          <box>
-            <size>0.0339686 0.060339 0.0468981</size>
-          </box>
-          <xacro:material_abb_yellow />
-        </geometry>
+        <xacro:material_abb_yellow />
       </collision>
     </link>
@@ -272,15 +77,12 @@
       <visual name="link_5">
         <geometry>
-          <mesh filename="package://abb_crb1100_support/meshes/crb1100_4_58/link_5.dae"/>
+          <mesh filename="package://abb_crb1100_support/meshes/crb1100_4_58/link_5.stl"/>
           <xacro:material_abb_white />
         </geometry>
       </visual>
-      <collision name="Link4_Cylinder011">
+      <collision name="collision">
         <pose>0.324441 0.0 0.617 1.5708 0.0 -1.5708</pose>
         <geometry>
-          <cylinder>
-            <length>0.0780414</length>
-            <radius>0.0353863</radius>
-          </cylinder>
+          <mesh filename="package://abb_crb1100_support/meshes/crb1100_4_58/link_5.stl"/>
           <xacro:material_abb_yellow />
         </geometry>
@@ -290,5 +92,5 @@
       <visual name="link_6">
         <geometry>
-          <mesh filename="package://abb_crb1100_support/meshes/crb1100_4_58/link_6.dae"/>
+          <mesh filename="package://abb_crb1100_support/meshes/crb1100_4_58/link_6.stl"/>
           <xacro:material_abb_white />
         </geometry>
@@ -296,5 +98,5 @@
       <collision name="Link4_Cylinder011">
         <geometry>
-          <mesh filename="package://abb_crb1100_support/meshes/crb1100_4_58/link_6.dae"/>
+          <mesh filename="package://abb_crb1100_support/meshes/crb1100_4_58/link_6.stl"/>
           <xacro:material_abb_yellow />
         </geometry>

Commit message: Go back to collider boxes
Signed-off-by: Yadunund <yadunund@openrobotics.org>

File: robot_specific_config/abb_crb1100_support/urdf/crb1100_4_58_macro.xacro (robot description, xacro)
@@ -11,7 +11,43 @@
         <xacro:material_abb_white />
       </visual>
-      <collision name"collision">
-        <geometry>
-          <mesh filename="package://abb_crb1100_support/meshes/crb1100_4_58/base_link.stl"/>
+      <collision name="Base_Box001">
+        <pose>-0.00780786 0.000316538 0.006 0.0 0.0 0.0</pose>
+        <geometry>
+          <box>
+            <size>0.174 0.158 0.012</size>
+          </box>
+        </geometry>
+      </collision>
+      <collision name="Base_Cylinder001">
+        <pose>0.0 0.0 0.0728 0.0 0.0 0.0</pose>
+        <geometry>
+          <cylinder>
+            <length>0.1456</length>
+            <radius>0.0719661</radius>
+          </cylinder>
+        </geometry>
+      </collision>
+      <collision name="Base_Box002">
+        <pose>-0.079843 0.0 0.0749219 1.5708 0.0 -1.5708</pose>
+        <geometry>
+          <box>
+            <size>0.110911 0.139336 0.0984126</size>
+          </box>
+        </geometry>
+      </collision>
+      <collision name="Base_Box003">
+        <pose>-0.13596 0.0 0.103253 1.5708 0.0 -1.5708</pose>
+        <geometry>
+          <box>
+            <size>0.0964925 0.0459809 0.0285397</size>
+          </box>
+        </geometry>
+      </collision>
+      <collision name="Base_Box004">
+        <pose>-0.131965 0.0 0.045724 1.5708 0.0 -1.5708</pose>
+        <geometry>
+          <box>
+            <size>0.0635693 0.0710773 0.0205486</size>
+          </box>
         </geometry>
         <xacro:material_abb_yellow />
@@ -25,7 +61,44 @@
         <xacro:material_abb_white />
       </visual>
-      <collision name="collision">
-        <geometry>
-          <mesh filename="package://abb_crb1100_support/meshes/crb1100_4_58/link_1.stl"/>
+      <collision name="Link1_Cylinder002">
+        <pose>0.0 0.0 0.180716 0.0 0.0 0.0</pose>
+        <geometry>
+          <cylinder>
+            <length>0.0695336</length>
+            <radius>0.0880028</radius>
+          </cylinder>
+        </geometry>
+      </collision>
+      <collision name="Link1_Cylinder003">
+        <pose>-2.53022e-05 -0.000703648 0.327248 1.5708 0.0 0.0</pose>
+        <geometry>
+          <cylinder>
+            <length>0.184809</length>
+            <radius>0.0517311</radius>
+          </cylinder>
+        </geometry>
+      </collision>
+      <collision name="Link1_Box005">
+        <pose>0.00740042 -0.0015163 0.268765 0.0 -0.131547 0.0</pose>
+        <geometry>
+          <box>
+            <size>0.0988751 0.182474 0.12116</size>
+          </box>
+        </geometry>
+      </collision>
+      <collision name="Link1_Box006">
+        <pose>-0.0321942 -0.0015163 0.218345 0.0 -0.213012 0.0</pose>
+        <geometry>
+          <box>
+            <size>0.0988751 0.178825 0.0508871</size>
+          </box>
+        </geometry>
+      </collision>
+      <collision name="Link1_Box007">
+        <pose>0.0360969 -0.00151631 0.209101 0.0 0.317913 0.0</pose>
+        <geometry>
+          <box>
+            <size>0.0988751 0.164519 0.0783661</size>
+          </box>
         </geometry>
         <xacro:material_abb_yellow />
@@ -40,6 +113,26 @@
       </visual>
       <collision name="Link2_Box008">
-        <geometry>
-          <mesh filename="package://abb_crb1100_support/meshes/crb1100_4_58/link_2.stl"/>
+        <pose>-0.0174075 0.0 0.423644 0.0 0.0 0.0</pose>
+        <geometry>
+          <box>
+            <size>0.0667305 0.0928778 0.198962</size>
+          </box>
+        </geometry>
+      </collision>
+      <collision name="Link2_Cylinder004">
+        <pose>-0.000196304 -0.000291631 0.606764 1.5708 0.0 0.0</pose>
+        <geometry>
+          <cylinder>
+            <length>0.178434</length>
+            <radius>0.0465957</radius>
+          </cylinder>
+        </geometry>
+      </collision>
+      <collision name="Link2_Box009">
+        <pose>-0.0103307 0.0 0.531581 0.0 0.01412 0.0</pose>
+        <geometry>
+          <box>
+            <size>0.0734036 0.176468 0.163149</size>
+          </box>
         </geometry>
         <xacro:material_abb_yellow />
@@ -53,7 +146,45 @@
         <xacro:material_abb_white />
       </visual>
-      <collision name="collision">
-        <geometry>
-          <mesh filename="package://abb_crb1100_support/meshes/crb1100_4_58/link_3.stl"/>
+      <collision name="Link3_Cylinder005">
+        <pose>-1.58772e-05 0.0 0.617021 1.5708 0.0 -1.5708</pose>
+        <geometry>
+          <cylinder>
+            <length>0.146229</length>
+            <radius>0.0454588</radius>
+          </cylinder>
+        </geometry>
+      </collision>
+      <collision name="Link3_Cylinder006">
+        <pose>0.000346811 -6.09569e-05 0.607321 1.5708 0.0 -1.19209e-07</pose>
+        <geometry>
+          <cylinder>
+            <length>0.0954674</length>
+            <radius>0.0454588</radius>
+          </cylinder>
+        </geometry>
+      </collision>
+      <collision name="Link3_Cylinder007">
+        <pose>-1.58772e-05 0.0 0.589443 1.5708 0.0 -1.5708</pose>
+        <geometry>
+          <cylinder>
+            <length>0.146229</length>
+            <radius>0.0454588</radius>
+          </cylinder>
+        </geometry>
+      </collision>
+      <collision name="Link3_Box010">
+        <pose>-0.0169157 0.0 0.653855 0.0 0.0 0.0</pose>
+        <geometry>
+          <box>
+            <size>0.018736 0.0498875 0.0203162</size>
+          </box>
+        </geometry>
+      </collision>
+      <collision name="Link3_Box011">
+        <pose>-0.0289604 -0.0174093 0.565988 0.0 0.0 0.0</pose>
+        <geometry>
+          <box>
+            <size>0.018736 0.0498875 0.0262079</size>
+          </box>
         </geometry>
         <xacro:material_abb_yellow />
@@ -67,7 +198,53 @@
         <xacro:material_abb_white />
       </visual>
-      <collision name="collision">
-        <geometry>
-          <mesh filename="package://abb_crb1100_support/meshes/crb1100_4_58/link_4.stl"/>
+      <collision name="Link4_Cylinder008">
+        <pose>0.15523 0.0 0.617 1.5708 0.0 1.5708</pose>
+        <geometry>
+          <cylinder>
+            <length>0.163185</length>
+            <radius>0.0452081</radius>
+          </cylinder>
+        </geometry>
+      </collision>
+      <collision name="Link4_Cylinder009">
+        <pose>0.3 0.0 0.617 1.5708 0.0 -1.74846e-07</pose>
+        <geometry>
+          <cylinder>
+            <length>0.102</length>
+            <radius>0.038</radius>
+          </cylinder>
+        </geometry>
+      </collision>
+      <collision name="Link4_Cylinder010">
+        <pose>0.179 0.0 0.617 1.5708 0.0 -1.74846e-07</pose>
+        <geometry>
+          <cylinder>
+            <length>0.102</length>
+            <radius>0.038</radius>
+          </cylinder>
+        </geometry>
+      </collision>
+      <collision name="Link4_Box012">
+        <pose>0.239561 0.0 0.617 0.0 0.0 0.0</pose>
+        <geometry>
+          <box>
+            <size>0.12 0.102032 0.076</size>
+          </box>
+        </geometry>
+      </collision>
+      <collision name="Link4_Box013">
+        <pose>0.154738 0.0 0.649546 0.0 -0.436332 0.0</pose>
+        <geometry>
+          <box>
+            <size>0.0893911 0.0609485 0.0468981</size>
+          </box>
+        </geometry>
+      </collision>
+      <collision name="Link4_Box014">
+        <pose>0.203204 0.0 0.647963 0.0 0.0 0.0</pose>
+        <geometry>
+          <box>
+            <size>0.0339686 0.060339 0.0468981</size>
+          </box>
         </geometry>
         <xacro:material_abb_yellow />
@@ -78,13 +255,16 @@
         <geometry>
           <mesh filename="package://abb_crb1100_support/meshes/crb1100_4_58/link_5.stl"/>
-          <xacro:material_abb_white />
-        </geometry>
-      </visual>
-      <collision name="collision">
+        </geometry>
+        <xacro:material_abb_white />
+      </visual>
+      <collision name="Link4_Cylinder011">
         <pose>0.324441 0.0 0.617 1.5708 0.0 -1.5708</pose>
         <geometry>
-          <mesh filename="package://abb_crb1100_support/meshes/crb1100_4_58/link_5.stl"/>
-          <xacro:material_abb_yellow />
-        </geometry>
+          <cylinder>
+            <length>0.0780414</length>
+            <radius>0.0353863</radius>
+          </cylinder>
+        </geometry>
+        <xacro:material_abb_yellow />
       </collision>
     </link>
@@ -93,6 +273,6 @@
         <geometry>
           <mesh filename="package://abb_crb1100_support/meshes/crb1100_4_58/link_6.stl"/>
-          <xacro:material_abb_white />
-        </geometry>
+        </geometry>
+        <xacro:material_abb_white />
       </visual>
       <collision name="Link4_Cylinder011">
