Commit message: Include ros2_control xacro
Signed-off-by: Yadunund <yadunund@openrobotics.org>

File: robot_specific_config/abb_crb1100_support/urdf/crb1100_4_58.xacro (robot description, xacro)
@@ -7,6 +7,17 @@
   <xacro:arg name="rws_port" default="80"/>
   <xacro:property name="rws_port" value="$(arg rws_port)"/>
+  <xacro:arg name="configure_via_rws" default="false"/>
+  <xacro:property name="configure_via_rws" value="$(arg configure_via_rws)"/>
   <!-- Robot description -->
   <xacro:include filename="$(find abb_crb1100_support)/urdf/crb1100_4_58_macro.xacro"/>
   <xacro:abb_crb1100_4_58 prefix=""/>
+  <!-- ros2_control -->
+  <xacro:include filename="$(find abb_crb1100_support)/urdf/crb1100.ros2_control.xacro" />
+  <xacro:abb_ros2_control
+    name="ABBMultiInterfaceHardware"
+    prefix=""
+    use_fake_hardware="${use_fake_hardware}"
+    rws_ip="${rws_ip}"
+    rws_port="${rws_port}"
+    configure_via_rws="${configure_via_rws}"/>
 </robot>
